File: MiniDelay v1.0/MiniDelay/MiniDelay.kicad_sch (KiCad schematic)
At the start: 53 parts, among them J1 IDC_2x05, U1 TL074, U2 PT2399, U3 L7805

Commit message: Added part descriptions
Parts:
- C1, C11, C13, C17, C2, C3, C4, C8, C9: Part Description (none) -> Multilayer Ceramic Capacitors MLCC - SMD/SMT 50 V 0.1uF X7R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
- C10, C12, C15, C19: Part Description (none) -> Multilayer Ceramic Capacitors MLCC - SMD/SMT 50V 2200pF C0G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
- C14: Part Description (none) -> Multilayer Ceramic Capacitors MLCC - SMD/SMT 25V 0.33uF X7R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
- C16: Part Description (none) -> Multilayer Ceramic Capacitors MLCC - SMD/SMT 100 V 0.015 uF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
- C18, C7: Part Description (none) -> Multilayer Ceramic Capacitors MLCC - SMD/SMT 0603 50VDC 1uF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
- C20: Part Description (none) -> Multilayer Ceramic Capacitors MLCC - SMD/SMT 50V 4700pF X7R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
- C21: Part Description (none) -> Multilayer Ceramic Capacitors MLCC - SMD/SMT 50V 0.01uF X7R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
- C22: Part Description (none) -> Multilayer Ceramic Capacitors MLCC - SMD/SMT 50 V 68 pF C0G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
- C5: Part Description (none) -> Multilayer Ceramic Capacitors MLCC - SMD/SMT .22UF 50V 10% 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
- C6: Part Description (none) -> Multilayer Ceramic Capacitors MLCC - SMD/SMT 50 V 47 pF C0G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
- D1: Part Description (none) -> 3.0mm Round Through Hole LED
- J1: Package (none) -> Straight,P=2.54mm; Part Description (none) -> IDC Connector 2x05 2.54mm Pitch Straight
- LEVEL1, REPEATS1: Package (none) -> RD901F
- R1, R16: Part Description (none) -> Thick Film Resistors - SMD 1 MOhms 100mW 0603 1%
- R10, R11, R12, R13, R14, R15, R2, R4, R8: Part Description (none) -> Thick Film Resistors - SMD 10 kOhms 100mW 0603 1% AEC-Q200
- R17, R20, R21, R3, R6: Part Description (none) -> Thick Film Resistors - SMD 100 kOhms 100mW 0603 1%
- R18: Part Description (none) -> Thick Film Resistors - SMD 68 kOhms 100mW 0603 1%
- R19, R7: Part Description (none) -> Thick Film Resistors - SMD 20 kOhms 100mW 0603 1%
- R5: Part Description (none) -> Thick Film Resistors - SMD 2.7 kOhms 100mW 0603 1%
- R9: Part Description (none) -> Thick Film Resistors - SMD 1 kOhms 100mW 0603 1%
- TIME1: Manufacturers Part Number RD901F-40-15F-B100K -> RD901F-40-15R1-B100K; Mfg # RD901F-40-15F-B100K -> RD901F-40-15R1-B100K; Package (none) -> RD901F; Part Description 100K OHM Linear Taper Potentiometer D Shaft PCB 9mm -> 100K OHM Linear Taper Potentiometer Round Shaft PCB 9mm
- U1: Part Description (none) -> Operational Amplifiers - Op Amps Quad Low Noise JFET
- U2: Part Description (none) -> SOP-16_150mil Audio Interface ICs ROHS
- U3: Part Description (none) -> 62dB@(120Hz) 1.5A 2V@(1A) Fixed 5V~5V Positive 1 35V TO-252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
